File: gsa-lib.kicad_sch (KiCad schematic)
At the start: 60 parts, among them J1 CONN-1, J2 CONN-2, J3 CONN-4, J4 SKT-2, J5 CONN-3, J6 CONN-5, J7 SKT-3, K1 RELAY-SPDT, K2 RELAY-DPDT, Q1 NPN, Q2 PNP, Q3 NFET, Q4 PFET, Q5 NMOS-D, Q6 PMOS-D, Q7 NMOS-E, Q8 PMOS-E, SW1 SW-PUSH, SW2 SW-SPST, SW3 SW-DPST, SW4 SW-DPDT, SW5 SW-SPDT, SW6 SW-SP2T, SW7 SW-SP3T, T1 XFRMR, T2 XFRMR-CTR, T3 XFRMR-DUAL, U1 40106, U10 LM1876, U11 LM78XX, U12 LM79XX, U13 LM317, U14 LM377, U15 TDA2009, U16 NE555, U2 4017, U3 LM386, U4 TBA820M, U5 4093, U6 4066, U7 LM1875, U8 OPAMP, U9 741, X1 LINK

Commit message: Some renaming
Parts:
- added Q9: UJT, symbol GSA:UJT
Changed lines of the file:
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@@
 	(title_block
 		(title "GSA Schematic Library")
-		(date "May  2020")
-		(rev "1.1.0")
+		(date "Feb 2026")
+		(rev "1.2.0")
 		(company "Gemstone Amplification")
-		(comment 1 "© Tim Baldwin 2016,2020")
+		(comment 1 "© Tim Baldwin 2016,2026")
 		(comment 4 "Schematic Symbols")
 	)
@@
 	(symbol
 		(lib_id "gsa:NMOS-D")
-		(at 57.15 88.9 0)
+		(at 63.5 88.9 0)
 		(unit 1)
 		(exclude_from_sim no)
@@
 		(dnp no)
 		(property "Reference" "Q5"
-			(at 61.976 85.09 0)
+			(at 68.326 85.09 0)
 			(effects
 				(font
@@
 		)
 		(property "Value" "NMOS-D"
-			(at 65.278 92.71 0)
+			(at 71.628 92.71 0)
 			(effects
 				(font
@@
 		)
 		(property "Footprint" ""
-			(at 57.15 88.9 0)
+			(at 63.5 88.9 0)
 			(effects
 				(font
@@
 		)
 		(property "Datasheet" ""
-			(at 57.15 88.9 0)
+			(at 63.5 88.9 0)
 			(effects
 				(font
@@
 		)
 		(property "Description" ""
-			(at 57.15 88.9 0)
+			(at 63.5 88.9 0)
 			(effects
 				(font
@@
 	(symbol
 		(lib_id "gsa:NMOS-E")
-		(at 76.2 88.9 0)
+		(at 81.28 88.9 0)
 		(unit 1)
 		(exclude_from_sim no)
@@
 		(dnp no)
 		(property "Reference" "Q7"
-			(at 81.026 85.09 0)
+			(at 86.106 85.09 0)
 			(effects
 				(font
@@
 		)
 		(property "Value" "NMOS-E"
-			(at 84.328 92.71 0)
+			(at 89.408 92.71 0)
 			(effects
 				(font
@@
 		)
 		(property "Footprint" ""
-			(at 76.2 88.9 0)
+			(at 81.28 88.9 0)
 			(effects
 				(font
@@
 		)
 		(property "Datasheet" ""
-			(at 76.2 88.9 0)
+			(at 81.28 88.9 0)
 			(effects
 				(font
@@
 		)
 		(property "Description" ""
-			(at 76.2 88.9 0)
+			(at 81.28 88.9 0)
 			(effects
 				(font
@@
 	(symbol
 		(lib_id "gsa:PMOS-D")
-		(at 57.15 101.6 0)
+		(at 63.5 101.6 0)
 		(unit 1)
 		(exclude_from_sim no)
@@
 		(dnp no)
 		(property "Reference" "Q6"
-			(at 61.976 97.79 0)
+			(at 68.326 97.79 0)
 			(effects
 				(font
@@
 		)
 		(property "Value" "PMOS-D"
-			(at 65.278 105.41 0)
+			(at 71.628 105.41 0)
 			(effects
 				(font
@@
 		)
 		(property "Footprint" ""
-			(at 57.15 101.6 0)
+			(at 63.5 101.6 0)
 			(effects
 				(font
@@
 		)
 		(property "Datasheet" ""
-			(at 57.15 101.6 0)
+			(at 63.5 101.6 0)
 			(effects
 				(font
@@
 		)
 		(property "Description" ""
-			(at 57.15 101.6 0)
+			(at 63.5 101.6 0)
 			(effects
 				(font
@@
 	(symbol
 		(lib_id "gsa:PMOS-E")
-		(at 76.2 101.6 0)
+		(at 81.28 101.6 0)
 		(unit 1)
 		(exclude_from_sim no)
@@
 		(dnp no)
 		(property "Reference" "Q8"
-			(at 81.026 97.79 0)
+			(at 86.106 97.79 0)
 			(effects
 				(font
@@
 		)
 		(property "Value" "PMOS-E"
-			(at 84.328 105.41 0)
+			(at 89.408 105.41 0)
 			(effects
 				(font
@@
 		)
 		(property "Footprint" ""
-			(at 76.2 101.6 0)
+			(at 81.28 101.6 0)
 			(effects
 				(font
@@
 		)
 		(property "Datasheet" ""
-			(at 76.2 101.6 0)
+			(at 81.28 101.6 0)
 			(effects
 				(font
@@
 		)
 		(property "Description" ""
-			(at 76.2 101.6 0)
+			(at 81.28 101.6 0)
 			(effects
 				(font
@@
 	(symbol
 		(lib_id "gsa:NFET")
-		(at 40.64 88.9 0)
+		(at 38.1 88.9 0)
 		(unit 1)
 		(exclude_from_sim no)
@@
 		(dnp no)
 		(property "Reference" "Q3"
-			(at 44.8056 87.7316 0)
+			(at 42.2656 87.7316 0)
 			(effects
 				(font
@@
 		)
 		(property "Value" "NFET"
-			(at 43.18 92.71 0)
+			(at 40.64 92.71 0)
 			(effects
 				(font
@@
 		)
 		(property "Footprint" ""
-			(at 40.64 88.9 0)
+			(at 38.1 88.9 0)
 			(effects
 				(font
@@
 		)
 		(property "Datasheet" ""
-			(at 40.64 88.9 0)
+			(at 38.1 88.9 0)
 			(effects
 				(font
@@
 		)
 		(property "Description" ""
-			(at 40.64 88.9 0)
+			(at 38.1 88.9 0)
 			(effects
 				(font
@@
 	(symbol
 		(lib_id "gsa:PFET")
-		(at 40.64 101.6 0)
+		(at 38.1 101.6 0)
 		(unit 1)
 		(exclude_from_sim no)
@@
 		(dnp no)
 		(property "Reference" "Q4"
-			(at 44.8056 100.4316 0)
+			(at 42.2656 100.4316 0)
 			(effects
 				(font
@@
 		)
 		(property "Value" "PFET"
-			(at 43.18 105.41 0)
+			(at 40.64 105.41 0)
 			(effects
 				(font
@@
 		)
 		(property "Footprint" ""
-			(at 40.64 101.6 0)
+			(at 38.1 101.6 0)
 			(effects
 				(font
@@
 		)
 		(property "Datasheet" ""
-			(at 40.64 101.6 0)
+			(at 38.1 101.6 0)
 			(effects
 				(font
@@
 		)
 		(property "Description" ""
-			(at 40.64 101.6 0)
+			(at 38.1 101.6 0)
 			(effects
 				(font
@@
 					(unit 1)
 				)
+			)
+		)
+	)
+	(symbol
+		(lib_id "GSA:UJT")
+		(at 50.8 88.9 0)
+		(unit 1)
+		(exclude_from_sim no)
+		(in_bom yes)
+		(on_board yes)
+		(dnp no)
+		(property "Reference" "Q9"
+			(at 55.88 87.6299 0)
+			(effects
+				(font
+					(size 1.27 1.27)
+				)
+				(justify left)
+				(hide yes)
+			)
+		)
+		(property "Value" "UJT"
+			(at 53.848 92.71 0)
+			(effects
+				(font
+					(size 1.27 1.27)
+				)
+				(justify left)
+			)
+		)
+		(property "Footprint" ""
+			(at 50.8 88.9 0)
+			(effects
+				(font
+					(size 1.27 1.27)
+				)
+				(hide yes)
+			)
+		)
+		(property "Datasheet" ""
+			(at 50.8 88.9 0)
+			(effects
+				(font
+					(size 1.27 1.27)
+				)
+				(hide yes)
+			)
+		)
+		(property "Description" ""
+			(at 50.8 88.9 0)
+			(effects
+				(font
+					(size 1.27 1.27)
+				)
+				(hide yes)
+			)
+		)
+		(pin "b1"
+		)
+		(pin "e"
+		)
+		(pin "b2"
+		)
+		(instances
+			(project ""
+				(path "/c14e7037-c8f8-4fad-93b5-84a1fe31f353"
+					(reference "Q9")
+					(unit 1)
+				)
