File: gsa-lib.kicad_pcb (KiCad board)
At the start: 2 copper layers, 115 parts

Commit message: KiCad v10 and add RES-T and PAD-T
Parts:
- added REF**: PAD-T, GSA:PAD-T, F.Cu at (70.0, 31.5)
- added Resistor/Trimmer: RES-T, GSA:RES-T, F.Cu at (124.0, 49.0)
- moved 10mm 18.0 mm to (110.5, 32.5)
- moved 2.5mm 18.0 mm to (91.7, 32.4)
- moved 5mm 18.0 mm to (99.3, 32.4)
Other:
- board text added: "Test Pads"
